Commit message: add scout mini urdf

File: src/my_robot_description/urdf/scout_mini_wheel.xacro (robot description, xacro)
@@ -11,5 +11,5 @@
                 <origin xyz="0 0 0" rpy="0 0 0" />
                 <geometry>
-                    <mesh filename="package://scout_description/meshes/wheel.dae" />
+                    <mesh filename="file:///home/scoutmini/workspace/indoor-nav-system/src/my_robot_description/meshes/wheel.dae" />
                 </geometry>
             </visual>
@@ -20,5 +20,5 @@
               <geometry>
                 <mesh
-                  filename="package://scout_description/meshes/wheel.dae" />
+                  filename="file:///home/scoutmini/workspace/indoor-nav-system/src/my_robot_description/meshes/wheel.dae" />
               </geometry>
             </collision>
