Commit message: add lidar urdf

File: src/my_robot_description/urdf/scout_mini.urdf.xacro (robot description, xacro)
@@ -170,3 +170,66 @@
     <!-- <xacro:include filename="$(find my_robot_description)/urdf/RS16.urdf.xacro"/>
     <xacro:RS16 origin="0 0 0 0 0 0"  /> -->
+  <xacro:property name="M_PI" value="3.1415926535897931" />
+  <xacro:macro name="RS-16" params="*origin parent:=base_link name:=robosense topic:=/robosense_points hz:=20 lasers:=16 samples:=900 collision_range:=0.4 min_range:=0.4 max_range:=150.0 noise:=0.008 min_angle:=-${M_PI} max_angle:=${M_PI} min_angle_vertical:=-${15.0*M_PI/180.0} max_angle_vertical:=-${15.0*M_PI/180.0} gpu:=false">
+    <joint name="${name}_base_mount_joint" type="fixed">
+      <xacro:insert_block name="origin" />
+      <parent link="${parent}"/>
+      <child link="${name}_base_link"/>
+    </joint>
+    <link name="${name}_base_link">
+      <inertial>
+        <mass value="0.87"/>
+        <origin xyz="0 0 0"/>
+        <inertia ixx="0.001094695" ixy="0" ixz="0"
+          iyy="0.001094695" iyz="0"
+          izz="0.001245079"/>
+      </inertial>
+      <visual>
+        <origin rpy="-1.5707 0 0" xyz="0 0 0"/>
+        <geometry>
+          <mesh filename="file:///home/scoutmini/workspace/indoor-nav-system/src/my_robot_description/meshes/robosense_16.dae" />
+        </geometry>
+      </visual>
+      <collision>
+        <origin rpy="0 0 0" xyz="0 0 0"/>
+        <geometry>
+          <cylinder radius="0.0535" length="0.0817"/>
+        </geometry>
+      </collision>
+    </link>
+    <joint name="${name}_base_scan_joint" type="fixed" >
+      <origin xyz="0 0 0.039" rpy="0 0 0" />
+      <parent link="${name}_base_link" />
+      <child link="${name}"/>
+    </joint>
+    <link name="${name}">
+      <inertial>
+        <mass value="0.01"/>
+        <origin xyz="0 0 0"/>
+        <inertia ixx="1e-7" ixy="0" ixz="0" iyy="1e-7" iyz="0" izz="1e-7"/>
+      </inertial>
+    </link>
+    <xacro:include filename="$(find my_robot_description)/urdf/robosense_lidar_sensor.gazebo"/>
+    <xacro:robosense_lidar_sensor
+      name="${name}"
+      topic="${topic}"
+      rate="${hz}"
+      lasers="${lasers}"
+      samples="${samples}"
+      collision_range="${collision_range}"
+      min_range="${min_range}"
+      max_range="${max_range}"
+      noise="${noise}"
+      min_angle="${min_angle}"
+      max_angle="${max_angle}"
+      min_angle_vertical="${min_angle_vertical}"
+      max_angle_vertical="${max_angle_vertical}"
+      gpu="${gpu}" />
+    </xacro:macro>
+    <xacro:arg name="gpu" default="false"/>
+    <xacro:property name="gpu" value="$(arg gpu)" />
+    <!-- <xacro:include filename="$(find my_robot_description)/urdf/RS-16.urdf.xacro"/> -->
+    <xacro:RS-16 parent="base_link" name="robosense" topic="/rs_points" hz="20" samples="900" gpu="${gpu}">
+        <origin xyz="0 0 0.4" rpy="0 0 0" />
+    </xacro:RS-16>
 </robot>

Commit message: add 2d lidar

File: src/my_robot_description/urdf/scout_mini.urdf.xacro (robot description, xacro)
@@ -92,4 +92,5 @@
         </plugin>
     </gazebo>
+    <xacro:include filename="$(find my_robot_description)/urdf/lidar2d.xacro" />
     <!-- kp spring constant, kd damping constant -->
     <!-- <gazebo>
@@ -170,5 +171,5 @@
     <!-- <xacro:include filename="$(find my_robot_description)/urdf/RS16.urdf.xacro"/>
     <xacro:RS16 origin="0 0 0 0 0 0"  /> -->
-  <xacro:property name="M_PI" value="3.1415926535897931" />
+  <!-- <xacro:property name="M_PI" value="3.1415926535897931" />
   <xacro:macro name="RS-16" params="*origin parent:=base_link name:=robosense topic:=/robosense_points hz:=20 lasers:=16 samples:=900 collision_range:=0.4 min_range:=0.4 max_range:=150.0 noise:=0.008 min_angle:=-${M_PI} max_angle:=${M_PI} min_angle_vertical:=-${15.0*M_PI/180.0} max_angle_vertical:=-${15.0*M_PI/180.0} gpu:=false">
     <joint name="${name}_base_mount_joint" type="fixed">
@@ -229,7 +230,6 @@
     <xacro:arg name="gpu" default="false"/>
     <xacro:property name="gpu" value="$(arg gpu)" />
-    <!-- <xacro:include filename="$(find my_robot_description)/urdf/RS-16.urdf.xacro"/> -->
     <xacro:RS-16 parent="base_link" name="robosense" topic="/rs_points" hz="20" samples="900" gpu="${gpu}">
         <origin xyz="0 0 0.4" rpy="0 0 0" />
-    </xacro:RS-16>
+    </xacro:RS-16> -->
 </robot>
