Commit message: slam_tool map works

File: src/my_robot_description/description/gazebo_control.xacro (robot description, xacro)
@@ -3,10 +3,10 @@
     <gazebo>
         <plugin name="diff_drive" filename="libgazebo_ros_diff_drive.so">
-            <!-- Wheel Information -->
+            <!-- Wheel Information
             <left_joint>left_wheel_joint</left_joint>
             <right_joint>right_wheel_joint</right_joint>
             <wheel_separation>0.297</wheel_separation>
-            <wheel_diameter>0.066</wheel_diameter>
-            <!-- Limits -->
+            <wheel_diameter>0.066</wheel_diameter> -->
+            Limits
             <max_wheel_torque>200</max_wheel_torque>
             <max_wheel_acceleration>10.0</max_wheel_acceleration>

File: src/my_robot_description/description/scout_mini.urdf.xacro (robot description, xacro)
@@ -3,3 +3,10 @@
     <xacro:include filename="scout_mini_core.xacro" />
     <!-- <xacro:include filename="$(find my_robot_description)/urdf/scout_wheel.gazebo" />  -->
+     <!-- Output -->
+            <!-- <odometry_frame>odom</odometry_frame>
+            <robot_base_frame>base_link</robot_base_frame> -->
+            <!-- <publish_odom>true</publish_odom>
+            <publish_odom_tf>true</publish_odom_tf>
+            <publish_wheel_tf>true</publish_wheel_tf>
+     -->
 </robot>

File: src/my_robot_description/description/scout_mini_core.xacro (robot description, xacro)
@@ -33,4 +33,11 @@
           </geometry>
         </collision>
+    </link>
+    <joint name="base_footprint_link" type="fixed">
+        <parent link="base_footprint" />
+        <child link="inertial_link" />
+        <origin xyz="0 0 0" rpy="0 0 0" />
+    </joint>
+    <link name="base_footprint">
     </link>
     <link name="inertial_link">
@@ -73,3 +80,6 @@
         <child link="rear_mount" />
     </joint>
+   <xacro:unless value="$(arg use_ros2_control)">
+        <xacro:include filename="gazebo_control.xacro" />
+    </xacro:unless>
 </robot>

File: src/my_robot_description/urdf/scout_mini.urdf.xacro (robot description, xacro)
@@ -233,3 +233,11 @@
         <origin xyz="0 0 0.4" rpy="0 0 0" />
     </xacro:RS-16> -->
+            <!-- Output -->
+            <plugin name="diff_drive" filename="libgazebo_ros_diff_drive.so">
+            <odometry_frame>odom</odometry_frame>
+            <robot_base_frame>base_link</robot_base_frame>
+            <publish_odom>true</publish_odom>
+            <publish_odom_tf>true</publish_odom_tf>
+            <publish_wheel_tf>true</publish_wheel_tf>
+            </plugin>
 </robot>
